File: hardware/alakol.kicad_pcb (KiCad board)
At the start: 4 copper layers, 78 x 56 mm, 116 parts, among them IC1 KSZ8081RNx, IC2 STM32H743VIT6, IC3 MS5607-02BA03, J1 CONN_01x08, J2 08B0-1X1T-06-F, J3 Side PCB, J4 Barrel_Jack_Switch, P1 SWD, Q1 BC817, Q2 BSS138BK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

Commit message: Hardware rev.1
Parts:
- added R45: 0Ω, agg:0402, F.Cu at (183.4, 110.5)
- added R46: 10kΩ, agg:0402, F.Cu at (161.0, 111.0)
- Y3: value SMD_XTAL -> SMD_XTAL_38.4_MHz
- moved C15 0.50 mm to (182.5, 118.0), turned to 270 degrees
Connections:
- IC2 pad 29: (no net) -> /PRESSURE_SCLK
- IC2 pad 42: (no net) -> Net-(IC2-Pad42)
- IC2 pad 89: /PRESSURE_SCLK -> /TRACESWO
- IC2 pad 94: (no net) -> /BOOT0
- P1 pad 6: Net-(P1-Pad6) -> /TRACESWO
- R29 pad 2: /PHY_MDC -> /PHY_MDIO
- R34 pad 2: GND -> 3v3
Routing:
- net /TRACESWO: track 0.00 -> 37.1 mm, vias 0 -> 1
- net /PRESSURE_SCLK: track 16.2 -> 30.6 mm
- net /BOOT0: track 0.00 -> 8.82 mm, vias 0 -> 2
- net /PHY_MDIO: track 19.4 -> 23.7 mm
- net 3v3: track 37.3 -> 40.3 mm
- net /PHY_MDC: track 27.0 -> 24.5 mm
- net Net-(IC2-Pad42): track 0.00 -> 2.30 mm
- net GND: track 69.0 -> 69.7 mm, vias 54 -> 52
Other:
- board text added: "Alakol"
- board text added: "Richard Meadows M0SBU 2020"
- board text added: "rev.1"
