File: hardware/alakol.sch (KiCad schematic (older format))
At the start: 116 parts, among them IC1 KSZ8081RNx, IC2 STM32H743VIT6, IC3 MS5607-02BA03, J1 CONN_01x08, J2 08B0-1X1T-06-F, J3 Side PCB, J4 Barrel_Jack_Switch, P1 SWD, Q1 BC817, Q2 BSS138BK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

Commit message: Hardware rev.1
Parts:
- added R45: 0Ω, agg:0402, symbol Device:R
- added R46: 10kΩ, agg:0402, symbol Device:R
- Y3: value SMD_XTAL -> SMD_XTAL_38.4_MHz
Connections:
- net 3v3: now also R34.2
- net GND: now also R45.2, R46.1; no longer R34.2
- net PHY_MDC: no longer R29.2
- net PHY_MDIO: now also R29.2
- net PRESSURE_SCLK: now also IC2.29 (PA5); no longer IC2.89 (PB3)
- net TRACESWO: now reaches P1.6 (SWO/TDO)
- net TRACESWO: now also IC2.89 (PB3)
- net at IC2.42 (PE12): now also R45.1
- net BOOT0: now reaches IC2.94 (BOOT0)
- net BOOT0: now also R46.2
Other:
- note added: "0b0001 = 1"
- note added: "HWVERSION"
- moved on the sheet: C1, C10, C11, C12, C13, C14, C15, C16, C17, C18, C19, C2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
